File: STM32 with Bluetooth/_autosave-STM32 with Bluetooth.kicad_sch (KiCad schematic)
At the start: 23 parts, among them U1 STM32WB55CCU6, X1 32KHz768, X2 32MHz

Commit message: Usb connector
Parts:
- added C17: 4u7, symbol Device:C
- added C18: 0p8, symbol Device:C
- added FLT1: DLF162500LT-5028A1, DLF162500LT-5028A1_Library:DLF162500LT-5028A1, symbol Stm32_Library:DLF162500LT-5028A1
- added J1: Conn_Coaxial, symbol Connector:Conn_Coaxial
- added J2: Conn_ARM_SWD_TagConnect_TC2030, Connector:Tag-Connect_TC2030-IDC-FP_2x03_P1.27mm_Vertical, symbol Connector:Conn_ARM_SWD_TagConnect_TC2030
- added J3: USB_C_Receptacle_USB2.0, symbol Connector:USB_C_Receptacle_USB2.0
- added R2, R3: R, symbol Device:R
- added SW1: SW_Push, symbol Switch:SW_Push
- added U2: USBLC6-2SC6, Package_TO_SOT_SMD:SOT-23-6, symbol Power_Protection:USBLC6-2SC6
Connections:
- net +3.3V: now also J2.1 (VCC)
- net GND: now also C17.2, C18.2, FLT1.2 (GND), FLT1.4 (GND), J1.2 (Ext), J2.5 (GND), J3.A1 (GND), J3.A12 (GND), J3.B1 (GND), J3.B12 (GND), J3.S1 (SHIELD), R2.2, U2.2 (GND)
- net at C16.1, L3.2: now also FLT1.1 (IN)
- net USB_D-: now reaches U1.37 (PA11)
- net USB_D-: now also U2.6 (I/O1)
- net USB_D+: now reaches U1.38 (PA12)
- net USB_D+: now also U2.4 (I/O2)
- net BOOT0: now reaches U1.4 (PH3)
- net BOOT0: now also C18.1, R2.1, R3.1
- net at U1.41 (PA14): now also J2.4 (SWCLK)
- net at U1.42 (PA15): now also J2.2 (SWDIO)
- net at U1.43 (PB3): now also J2.6 (SWO)
- net NRST: now reaches U1.7 (NRST)
- net NRST: now also C17.1, J2.3 (~{RESET})
- new net: R3.2, SW1.1
- new net: FLT1.3 (OUT), J1.1 (In)
- new net: J3.A7 (D-), J3.B7 (D-), U2.1 (I/O1)
- new net: J3.A6 (D+), J3.B6 (D+), U2.3 (I/O2)
- new net: J3.A4 (VBUS), J3.A9 (VBUS), J3.B4 (VBUS), J3.B9 (VBUS)
Other:
- moved on the sheet: C1, C10, C11, C12, C13, C14, C15, C16, C2, C3, C4, C5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

Commit message: final schematics
Parts:
- added C19, C20: 4u7, symbol Device:C
- added D1: LED, symbol Device:LED
- added J4: Conn_01x04, symbol Connector_Generic:Conn_01x04
- added R4, R5: 5K1, symbol Device:R
- added R6, R7, R8: 220, symbol Device:R
- added U3: MIC5365-3.3YD5, Package_TO_SOT_SMD:SOT-23-5, symbol Regulator_Linear:MIC5365-3.3YD5
- R2: value R -> 5K1
- R3: value R -> 100
Connections:
- net +3.3V: now also SW1.2, C20.1, J4.1 (Pin_1), U3.5 (VOUT)
- net GND: now also C19.2, C20.2, J4.4 (Pin_4), R4.2, R5.2, R8.1, U3.2 (GND)
- net at U2.5 (VBUS): now also J3.A4 (VBUS), J3.A9 (VBUS), J3.B4 (VBUS), J3.B9 (VBUS), C19.1, U3.1 (VIN), U3.3 (EN)
- net at J3.A5 (CC1): now also R5.1
- net at J3.B5 (CC2): now also R4.1
- net UART_TX: now reaches U1.11 (PA2)
- net UART_TX: now also R7.2
- net UART_RX: now reaches U1.12 (PA3)
- net UART_RX: now also R6.2
- net at U1.16 (PA7): now also D1.2 (A)
- new net: D1.1 (K), R8.2
- new net: J4.3 (Pin_3), R7.1
- new net: J4.2 (Pin_2), R6.1
- no-connect marks 0 -> 21
Other:
- note added: "5V TO 3.3V REGULATOR"
- note added: "BOOT0 SWITCH"
- note added: "RF AND U.FL CONNECTOR"
- note added: "STM32WB55CCU6 MCU"
- note added: "UART Header"
- note added: "USB C CONNECTION"
- title: (none) -> STM32WB55
- moved on the sheet: C15, C16, C18, FLT1, J1, J2, J3, L3, R2, R3, SW1, U2
