File: STM32 with Bluetooth/_autosave-STM32 with Bluetooth.kicad_sch (KiCad schematic)
At the start: 42 parts, among them J1 Conn_Coaxial, J2 USB_C_Receptacle_USB2.0, J3 Conn_ARM_SWD_TagConnect_TC2030, J4 Conn_01x04, SW1 SW_Push, U1 MIC5365-3.3YD5, U2 USBLC6-2SC6, U3 STM32WB55CCU6, X1 32MHz, X2 32KHz768

Commit message: pcb
Connections:
- no-connect marks 28 -> 27
Changed lines of the file:
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@@
   (no_connect (at 182.88 129.54))
   (no_connect (at 182.88 147.32))
-  (no_connect (at 142.24 84.455))
   (no_connect (at 182.88 142.24))
   (no_connect (at 182.88 167.64))
