File: STM32 with Bluetooth/STM32 with Bluetooth.kicad_sch (KiCad schematic)
At the start: 15 parts, among them U1 STM32WB55CCU6

Commit message: Electrical rule checked
Parts:
- added C1, C17, C2: 4u7, symbol Device:C
- added C15, C20: 0p8, symbol Device:C
- added C16: 0p3, symbol Device:C
- added C18, C19: C, symbol Device:C
- added D1: LED, symbol Device:LED
- added FLT1: DLF162500LT-5028A1, DLF162500LT-5028A1_Library:DLF162500LT-5028A1, symbol Stm32_Library:DLF162500LT-5028A1
- added J1: Conn_Coaxial, symbol Connector:Conn_Coaxial
- added J2: USB_C_Receptacle_USB2.0, symbol Connector:USB_C_Receptacle_USB2.0
- added J3: Conn_ARM_SWD_TagConnect_TC2030, Connector:Tag-Connect_TC2030-IDC-FP_2x03_P1.27mm_Vertical, symbol Connector:Conn_ARM_SWD_TagConnect_TC2030
- added J4: Conn_01x04, symbol Connector_Generic:Conn_01x04
- added L3: 2n7, symbol Device:L
- added R1: 0, symbol Device:R
- added R2, R6, R8: 220, symbol Device:R
- added R3, R4, R7: 5K1, symbol Device:R
- added R5: 100, symbol Device:R
- added SW1: SW_Push, symbol Switch:SW_Push
- added U1: MIC5365-3.3YD5, Package_TO_SOT_SMD:SOT-23-5, symbol Regulator_Linear:MIC5365-3.3YD5
- added U2: USBLC6-2SC6, Package_TO_SOT_SMD:SOT-23-6, symbol Power_Protection:USBLC6-2SC6
- added X1: 32MHz, symbol Device:Crystal_GND24
- added X2: 32KHz768, symbol Device:Crystal
- renumbered C4 to C10, C3 to C11, C2 to C12, C1 to C13, C12 to C14, C10 to C3, C11 to C4, C8 to C5, C9 to C6, C6 to C8, C5 to C9, U1 to U3
Connections:
- net +3.3V: now also C2.1, J3.1 (VCC), J4.1 (Pin_1), SW1.2, U1.5 (VOUT)
- net GND: now also C1.2, C15.2, C16.2, C17.2, C18.2, C19.2, C2.2, C20.2, FLT1.2 (GND), FLT1.4 (GND), J1.2 (Ext), J2.A1 (GND), J2.A12 (GND), J2.B1 (GND), J2.B12 (GND), J2.S1 (SHIELD), J3.5 (GND), J4.4 (Pin_4), R2.1, R3.2, R4.2, R7.2, U1.2 (GND), U2.2 (GND), X1.2, X1.4
- net UART_TX: now reaches U3.11 (PA2)
- net UART_TX: now also R8.2
- net UART_RX: now reaches U3.12 (PA3)
- net UART_RX: now also R6.2
- net at U3.16 (PA7): now also D1.2 (A)
- net LSE_IN: now reaches U3.2 (PC14)
- net LSE_IN: now also C19.1, X2.2
- net at U3.21 (RF1): now also C15.1, L3.1
- net HSE_OUT: now reaches U3.24 (OSC_OUT)
- net HSE_OUT: now also R1.1
- net HSE_IN: now reaches U3.25 (OSC_IN)
- net HSE_IN: now also X1.3
- net LSE_OUT: now reaches U3.3 (PC15)
- net LSE_OUT: now also C18.1, X2.1
- net USB_D-: now reaches U3.37 (PA11)
- net USB_D-: now also U2.6 (I/O1)
- net USB_D+: now reaches U3.38 (PA12)
- net USB_D+: now also U2.4 (I/O2)
- net BOOT0: now reaches U3.4 (PH3)
- net BOOT0: now also C20.1, R5.1, R7.1
- net at U3.41 (PA14): now also J3.4 (SWCLK)
- net at U3.42 (PA15): now also J3.2 (SWDIO)
- net at U3.43 (PB3): now also J3.6 (SWO)
- net NRST: now reaches U3.7 (NRST)
- net NRST: now also C17.1, J3.3 (~{RESET})
- net SMPSLX: no longer names the net of L1.1, U3.33 (VLXSMPS)
- new net: R5.2, SW1.1
- new net: D1.1 (K), R2.2
- new net: C16.1, FLT1.1 (IN), L3.2
- new net: FLT1.3 (OUT), J1.1 (In)
- new net: J4.3 (Pin_3), R8.1
- new net: J2.A7 (D-), J2.B7 (D-), U2.1 (I/O1)
- new net: J2.A6 (D+), J2.B6 (D+), U2.3 (I/O2)
- new net: C1.1, J2.A4 (VBUS), J2.A9 (VBUS), J2.B4 (VBUS), J2.B9 (VBUS), U1.1 (VIN), U1.3 (EN), U2.5 (VBUS)
- new net: J2.A5 (CC1), R4.1
- new net: J2.B5 (CC2), R3.1
- new net: R1.2, X1.1
- new net: J4.2 (Pin_2), R6.1
- no-connect marks 0 -> 21
Other:
- note added: "5V TO 3.3V REGULATOR"
- note added: "BOOT0 SWITCH"
- note added: "RF AND U.FL CONNECTOR"
- note added: "STM32WB55CCU6 MCU"
- note added: "UART Header"
- note added: "USB C CONNECTION"
- title: (none) -> STM32WB55
- moved on the sheet: C10, C11, C12, C13, C14, C3, C4, C5, C6, C7, C8, C9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

Commit message: componnent assignment
Parts:
- C1, C14, C17, C2, C5, C7: footprint (none) -> Capacitor_SMD:C_0603_1608Metric
- C10, C11, C12, C13, C15, C16, C18, C19, C3, C4, C6, C8, C9: footprint (none) -> Capacitor_SMD:C_0402_1005Metric
- C20: value 0p8 -> 100n; footprint (none) -> Capacitor_SMD:C_0402_1005Metric
- D1: footprint (none) -> LED_SMD:LED_0402_1005Metric
- J1: footprint (none) -> Connector_Coaxial:U.FL_Hirose_U.FL-R-SMT-1_Vertical
- J2: footprint (none) -> Connector_USB:USB_C_Receptacle_GCT_USB4105-xx-A_16P_TopMnt_Horizontal
- J4: footprint (none) -> Connector_Molex:Molex_PicoBlade_53048-0410_1x04_P1.25mm_Horizontal
- L1, L2, L3: footprint (none) -> Inductor_SMD:L_0402_1005Metric
- R1, R2, R3, R4, R5, R6, R7, R8: footprint (none) -> Resistor_SMD:R_0402_1005Metric
- SW1: footprint (none) -> Button_Switch_SMD:SW_SPST_CK_RS282G05A3
- X1: footprint (none) -> Crystal:Crystal_SMD_2016-4Pin_2.0x1.6mm
- X2: footprint (none) -> Crystal:Crystal_SMD_2012-2Pin_2.0x1.2mm
